File: HVPS_SMD/HVPS_SMD.sch (KiCad schematic (older format))
At the start: 20 parts, among them J1 CONN_01X02, J2 CONN_01X02, J3 CONN_01X02, Q1 AO4294, T1 WE-FLEX_ER11_5, U1 LM3478SOIC8

Commit message: Clean up silk screen and DRC smells
Parts:
- C1: symbol CP1 -> HVPS_SMD:CP1
- C2, C3, Cc1, Cs1: symbol C_Small -> HVPS_SMD:C_Small
- D1: symbol DIODE -> HVPS_SMD:DIODE
- J1, J2, J3: symbol CONN_01X02 -> HVPS_SMD:CONN_01X02
- Q1: symbol MOSFET_SO08 -> HVPS_SMD:MOSFET_SO08
- R1, R2, R3, R4, Rc1, Rf1, Rs1, Rsen1: symbol R_Small -> HVPS_SMD:R_Small
- T1: symbol WE-FLEX_ER11_5 -> HVPS_SMD:WE-FLEX_ER11_5
- U1: symbol LM3478SOIC8 -> HVPS_SMD:LM3478SOIC8
Connections:
- wire segments 62 -> 78
Changed lines of the file:
@@
-EESchema Schematic File Version 2
-LIBS:HVPS_SMD
-LIBS:power
-LIBS:device
-LIBS:transistors
-LIBS:conn
-LIBS:linear
-LIBS:regul
-LIBS:74xx
-LIBS:cmos4000
-LIBS:adc-dac
-LIBS:memory
-LIBS:xilinx
-LIBS:microcontrollers
-LIBS:dsp
-LIBS:microchip
-LIBS:analog_switches
-LIBS:motorola
-LIBS:texas
-LIBS:intel
-LIBS:audio
-LIBS:interface
-LIBS:digital-audio
-LIBS:philips
-LIBS:display
-LIBS:cypress
-LIBS:siliconi
-LIBS:opto
-LIBS:atmel
-LIBS:contrib
+EESchema Schematic File Version 4
 LIBS:HVPS_SMD-cache
-EELAYER 25 0
+EELAYER 26 0
 EELAYER END
 $Descr USLetter 11000 8500
@@
 $EndDescr
 $Comp
-L LM3478SOIC8 U1
+L HVPS_SMD:LM3478SOIC8 U1
 U 1 1 59C866DF
 P 4300 3500
@@
 $EndComp
 $Comp
-L WE-FLEX_ER11_5 T1
+L HVPS_SMD:WE-FLEX_ER11_5 T1
 U 1 1 59C9939D
 P 6650 2000
@@
 $EndComp
 $Comp
-L MOSFET_SO08 Q1
+L HVPS_SMD:MOSFET_SO08 Q1
 U 1 1 59C9950D
 P 5550 3300
@@
 Vin
 $Comp
-L GND #PWR01
+L HVPS_SMD:GND #PWR01
 U 1 1 59C99721
 P 4300 4300
@@
 $EndComp
 $Comp
-L GND #PWR02
+L HVPS_SMD:GND #PWR02
 U 1 1 59C9973B
 P 4000 4300
@@
 $EndComp
 $Comp
-L GND #PWR03
+L HVPS_SMD:GND #PWR03
 U 1 1 59C99755
 P 5650 4300
@@
 $EndComp
 $Comp
-L R_Small Rsen1
+L HVPS_SMD:R_Small Rsen1
 U 1 1 59C9976F
 P 5650 4050
@@
 $EndComp
 $Comp
-L C_Small C2
+L HVPS_SMD:C_Small C2
 U 1 1 59C997CF
 P 5400 4050
@@
 $EndComp
 $Comp
-L GND #PWR04
+L HVPS_SMD:GND #PWR04
 U 1 1 59C99800
 P 5400 4300
@@
 $EndComp
 $Comp
-L C_Small Cc1
+L HVPS_SMD:C_Small Cc1
 U 1 1 59C999FD
 P 3450 3900
@@
 $EndComp
 $Comp
-L R_Small Rc1
+L HVPS_SMD:R_Small Rc1
 U 1 1 59C99A42
 P 3450 4150
@@
 $EndComp
 $Comp
-L GND #PWR05
+L HVPS_SMD:GND #PWR05
 U 1 1 59C99A69
 P 3450 4300
@@
 Vout
 $Comp
-L C_Small C3
+L HVPS_SMD:C_Small C3
 U 1 1 59C99D4C
 P 7550 1600
@@
 $EndComp
 $Comp
-L GND #PWR06
+L HVPS_SMD:GND #PWR06
 U 1 1 59C99D8F
 P 7550 2300
@@
 $EndComp
 $Comp
-L R_Small R2
+L HVPS_SMD:R_Small R2
 U 1 1 59C99FC3
 P 7000 3250
@@
 $EndComp
 $Comp
-L R_Small R3
+L HVPS_SMD:R_Small R3
 U 1 1 59C99FFA
 P 7000 4000
@@
 $EndComp
 $Comp
-L R_Small R4
+L HVPS_SMD:R_Small R4
 U 1 1 59C9A029
 P 7450 3400
@@
 Vadj
 $Comp
-L R_Small Rf1
+L HVPS_SMD:R_Small Rf1
 U 1 1 59C9A1BE
 P 3450 3400
@@
 $EndComp
 $Comp
-L GND #PWR07
+L HVPS_SMD:GND #PWR07
 U 1 1 59C9A23F
 P 7000 4300
@@
 $EndComp
 $Comp
-L R_Small Rs1
+L HVPS_SMD:R_Small Rs1
 U 1 1 59C9A340
 P 5150 2750
@@
 $EndComp
 $Comp
-L C_Small Cs1
+L HVPS_SMD:C_Small Cs1
 U 1 1 59C9A371
 P 5150 2400
@@
 $EndComp
 $Comp
-L CP1 C1
+L HVPS_SMD:CP1 C1
 U 1 1 59C9AACA
 P 2700 3450
@@
 $EndComp
 $Comp
-L GND #PWR08
+L HVPS_SMD:GND #PWR08
 U 1 1 59C9AB4B
 P 2700 4300
@@
 GND
 $Comp
-L CONN_01X02 J2
+L HVPS_SMD:CONN_01X02 J2
 U 1 1 59C9BAB8
 P 1700 2350
@@
 GND
 $Comp
-L GND #PWR09
+L HVPS_SMD:GND #PWR09
 U 1 1 59C9BC9B
 P 1700 3750
@@
 $EndComp
 $Comp
-L VCC #PWR010
+L HVPS_SMD:VCC #PWR010
 U 1 1 59C9BCD3
 P 1950 3750
@@
 $EndComp
 $Comp
-L HT #PWR011
+L HVPS_SMD:HT #PWR011
 U 1 1 59C9BD0B
 P 2200 3750
@@
 	2100 1650 1900 1650
 Wire Wire Line
-	5650 1900 5650 3100
+	5650 1900 5650 3000
 Wire Wire Line
 	2700 3600 2700 4300
@@
 	5150 2100 5150 2300
 Wire Wire Line
-	7000 4100 7000 4300
+	7000 4100 7000 4200
 Wire Wire Line
 	7550 3400 8300 3400
@@
 	7350 3400 7000 3400
 Wire Wire Line
-	7000 3350 7000 3900
+	7000 3350 7000 3400
 Wire Wire Line
 	7000 2850 7000 2900
@@
 Connection ~ 7550 2100
 Wire Wire Line
-	7550 1700 7550 2300
+	7550 1700 7550 2100
 Connection ~ 7550 1400
 Wire Wire Line
 	7550 1400 7550 1500
 Wire Wire Line
-	7450 1400 8150 1400
+	7450 1400 7550 1400
 Wire Wire Line
 	3450 4250 3450 4300
@@
 Connection ~ 5650 3800
 Wire Wire Line
-	5000 3800 5650 3800
+	5000 3800 5400 3800
 Wire Wire Line
 	5650 4150 5650 4300
 Wire Wire Line
-	5650 3500 5650 3950
-Wire Wire Line
-	4300 2100 4300 3000
-Wire Wire Line
-	2500 2600 4300 2600
+	5650 3500 5650 3800
+Wire Wire Line
+	4300 2100 4300 2600
+Wire Wire Line
+	2500 2600 2700 2600
 Wire Wire Line
 	5000 3400 5450 3400
 $Comp
-L R_Small R1
+L HVPS_SMD:R_Small R1
 U 1 1 59C9CDD9
 P 7000 3000
@@
 	3350 3400 3250 3400
 $Comp
-L DIODE D1
+L HVPS_SMD:DIODE D1
 U 1 1 59CB0EFA
 P 7350 1400
@@
 	6450 1900 5650 1900
 Wire Wire Line
-	4300 2100 6450 2100
+	4300 2100 5150 2100
 Connection ~ 4300 2600
 Wire Wire Line
@@
 Connection ~ 8100 1400
 $Comp
-L CONN_01X02 J1
+L HVPS_SMD:CONN_01X02 J1
 U 1 1 59CC5EB0
 P 1700 1700
@@
 $EndComp
 $Comp
-L CONN_01X02 J3
+L HVPS_SMD:CONN_01X02 J3
 U 1 1 59CC5F0B
 P 2850 2150
@@
 	-1   0    0    1
 $EndComp
+Wire Wire Line
+	2700 2600 4300 2600
+Wire Wire Line
+	5150 2100 6450 2100
+Wire Wire Line
+	7000 3600 7000 3900
+Wire Wire Line
+	7000 3400 7000 3600
+Wire Wire Line
+	7550 2100 7550 2300
+Wire Wire Line
+	7550 1400 8100 1400
+Wire Wire Line
+	5400 3800 5650 3800
+Wire Wire Line
+	5650 3800 5650 3950
+Wire Wire Line
+	4300 2600 4300 3000
+Wire Wire Line
+	5650 3000 5650 3100
+Wire Wire Line
+	8100 1400 8150 1400
+$Comp
+L NixieClockMaster:PWR_FLAG #FLG0101
+U 1 1 5CA348AC
+P 4300 1950
+F 0 "#FLG0101" H 4300 2215 50  0000 C CNN
+F 1 "PWR_FLAG" H 4300 2124 50  0000 C CNN
+F 2 "" H 4300 1950 50  0001 C CNN
+F 3 "" H 4300 1950 50  0001 C CNN
+	1    4300 1950
+	1    0    0    -1
+$EndComp
+Wire Wire Line
+	4300 1950 4300 2100
+Connection ~ 4300 2100
+$Comp
+L NixieClockMaster:PWR_FLAG #FLG0102
+U 1 1 5CA362BF
+P 6700 4050
+F 0 "#FLG0102" H 6700 4315 50  0000 C CNN
+F 1 "PWR_FLAG" H 6700 4224 50  0000 C CNN
+F 2 "" H 6700 4050 50  0001 C CNN
+F 3 "" H 6700 4050 50  0001 C CNN
+	1    6700 4050
+	1    0    0    -1
+$EndComp
+Wire Wire Line
+	6700 4050 6700 4200
+Wire Wire Line
+	6700 4200 7000 4200
+Connection ~ 7000 4200
+Wire Wire Line
+	7000 4200 7000 4300
+$Comp
+L NixieClockMaster:PWR_FLAG #FLG0103
+U 1 1 5CA37C0D
+P 8100 1100
+F 0 "#FLG0103" H 8100 1365 50  0001 C CNN
+F 1 "PWR_FLAG" H 8100 1274 50  0000 C CNN
+F 2 "" H 8100 1100 50  0001 C CNN
+F 3 "" H 8100 1100 50  0001 C CNN
+	1    8100 1100
+	1    0    0    -1
+$EndComp
+Wire Wire Line
+	8100 1100 8100 1400
 $EndSCHEMATC
